File: luna.kicad_pcb (KiCad board)
At the start: 2 copper layers, 85 x 83.8 mm, 31 parts, among them J1 Conn_01x06_Male, J2 Conn_02x12_Top_Bottom, J3 Conn_01x02_Male, J4 Conn_01x02_Male, J5 Screw_Terminal_01x06, Q1 2N7002, Q2 2N7002, Q3 2N7002, Q4 DMN3404L, Q5 DMN3404L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

Commit message: Design in progress.
Parts:
- removed H1, H2, H3, H4: MountingHole_Pad, MountingHole:MountingHole_3.2mm_M3_Pad
- removed J4: Conn_01x02_Male, Connector_PinHeader_2.54mm:PinHeader_1x02_P2.54mm_Horizontal
- removed J5: Screw_Terminal_01x06, TerminalBlock_RND:TerminalBlock_RND_205-00291_1x06_P5.08mm_Horizontal
- removed Q5, Q6: DMN3404L, Package_TO_SOT_SMD:SOT-23
- added D3: D_Schottky, Diode_SMD:D_SOD-323_HandSoldering, F.Cu at (74.9, 55.3)
- added D4: D_Schottky, Diode_SMD:D_SOD-323_HandSoldering, F.Cu at (57.3, 75.6)
- added D5: LED_AGRB, custom:LED_STRIP_RGB, B.Cu at (29.0, 67.0)
- added D6: D_Schottky, Diode_SMD:D_SOD-323_HandSoldering, F.Cu at (69.8, 58.3)
- added D7: LED, custom:LED_STRIP, B.Cu at (40.0, 67.0)
- added L1: 6u5, Inductor_SMD:L_Bourns-SRN4018, F.Cu at (99.0, 52.0)
- added R7: 33k, Resistor_SMD:R_0805_2012Metric_Pad1.15x1.40mm_HandSolder, F.Cu at (103.0, 50.0)
- added R8: 10k, Resistor_SMD:R_0805_2012Metric_Pad1.15x1.40mm_HandSolder, F.Cu at (105.0, 48.0)
- added R9: 10k, Resistor_SMD:R_0805_2012Metric_Pad1.15x1.40mm_HandSolder, F.Cu at (79.1, 46.4)
- C1: value 10u -> 22u; moved to F.Cu
- C2, C3, C4, C6, D1, D2, R2, R5: moved to F.Cu
- C5: value 10u -> 1u; moved to F.Cu
- J1: value Conn_01x06_Male -> Conn_01x06_MountingPin; footprint Connector_PinHeader_2.54mm:PinHeader_1x06_P2.54mm_Horizontal -> Connector_FFC-FPC:Hirose_FH12-6S-0.5SH_1x06-1MP_P0.50mm_Horizontal
- J2: value Conn_02x12_Top_Bottom -> Conn_01x01; footprint Connector_Molex:Molex_Mini-Fit_Jr_5569-24A2_2x12_P4.20mm_Horizontal -> Connector_Wire:SolderWirePad_1x01_SMD_5x10mm
- J3: value Conn_01x02_Male -> Conn_01x01; footprint Connector_PinHeader_2.54mm:PinHeader_1x02_P2.54mm_Horizontal -> Connector_Wire:SolderWirePad_1x01_SMD_5x10mm
- Q1, Q2, Q3: value 2N7002 -> DMN3404L
- R1, R3: value 1k -> 10k; moved to F.Cu
- R4: value 10k -> 100k; moved to F.Cu
- R6: value 10k -> 47k; moved to F.Cu
- U1: value LD1117S33TR_SOT223 -> AP65111AWU; footprint Package_TO_SOT_SMD:SOT-223-3_TabPin2 -> Package_TO_SOT_SMD:TSOT-23-6; moved to F.Cu
- moved C1 72.6 mm to (98.0, 43.0), turned to 0 degrees
- moved R1 66.4 mm to (67.8, 67.6), turned to 0 degrees
- moved U1 64.5 mm to (99.0, 46.0)
- moved R3 54.6 mm to (79.1, 52.3), turned to 0 degrees
- moved R6 49.7 mm to (103.0, 46.0), turned to 270 degrees
- moved Q3 49.3 mm to (32.0, 62.0), turned to 0 degrees
- moved J1 47.3 mm to (28.0, 47.0), turned to 0 degrees
- moved C2 47.2 mm to (51.8, 75.8), turned to 0 degrees
- moved Q2 46.1 mm to (24.0, 61.0), turned to 0 degrees
- moved Q1 45.0 mm to (29.0, 59.0), turned to 0 degrees
- moved Q4 41.2 mm to (36.0, 60.0), turned to 0 degrees
- moved U2 36.6 mm to (32.0, 29.8), turned to 180 degrees
- moved R2 36.2 mm to (74.7, 58.3), turned to 0 degrees
- moved J2 35.9 mm to (59.0, 34.0), turned to 0 degrees
- moved C5 31.8 mm to (99.0, 49.0), turned to 0 degrees
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Connections:
- net DUMMY_LOAD renamed LED_W
- net Net-(J4-Pad2) renamed LED_B_OUT
- C1 pad 1: +5V -> +12V
- C2 pad 1: GND -> +12V
- C2 pad 2: +5V -> GND
- C3 pad 1: VDD -> +12V
- C4 pad 2: GNDPWR -> GND
- C5 pad 1: +12V -> Net-(C5-Pad1)
- C5 pad 2: GNDPWR -> Net-(C5-Pad2)
- C6 pad 2: GNDPWR -> GND
- D1 pad 2: LED_W1_OUT -> LED_R_OUT
- D2 pad 2: LED_W2_OUT -> LED_G_OUT
- J2 pad 1: Net-(J2-Pad1) -> +12V
- Q1 pad 1: VDD -> LED_R
- Q1 pad 2: RGB1 -> GND
- Q1 pad 3: Net-(J3-Pad2) -> LED_R_OUT
- Q2 pad 1: ~ON~ -> LED_G
- Q2 pad 3: Net-(J2-Pad16) -> LED_G_OUT
- Q3 pad 1: VDD -> LED_B
- Q3 pad 2: RGB2 -> GND
- Q4 pad 2: GNDPWR -> GND
- Q4 pad 3: DUMMY_LOAD_OUT -> Net-(D6-Pad2)
- R1 pad 1: +5V -> +12V
- R1 pad 2: Net-(J3-Pad2) -> LED_R_OUT
- R2 pad 1: ~ON~ -> +12V
- R2 pad 2: GND -> LED_G_OUT
- R3 pad 1: +5V -> +12V
- R4 pad 1: VDD -> Net-(R4-Pad1)
- R4 pad 2: EN -> +12V
- R5 pad 2: LED_W1_OUT -> Net-(D6-Pad2)
- R6 pad 1: +12V -> Net-(R6-Pad1)
- R6 pad 2: LED_W2_OUT -> Net-(R6-Pad2)
- U1 pad 1: GND -> +12V
- U1 pad 2: VDD -> GND
- U1 pad 3: +5V -> Net-(C5-Pad1)
- U2 pad 10: LED_W2 -> LED_G
- U2 pad 11: RGB1 -> LED_B
- U2 pad 12: RGB2 -> Net-(U2-Pad12)
- U2 pad 13: ~ON~ -> Net-(U2-Pad13)
- U2 pad 9: LED_W1 -> LED_R
Routing:
- net +5V: track 107.2 -> 0.00 mm
- net VDD: track 99.5 -> 0.00 mm
- net Net-(J2-Pad16): track 51.1 -> 0.00 mm, vias 1 -> 0
- net EN: track 44.4 -> 0.00 mm, vias 1 -> 0
- net RGB1: track 40.2 -> 0.00 mm
- net RGB2: track 34.4 -> 0.00 mm
- net LED_W2: track 30.3 -> 0.00 mm, vias 2 -> 0
- net LED_W: track 28.7 -> 0.00 mm, vias 2 -> 0
- net LED_W1: track 26.6 -> 0.00 mm, vias 2 -> 0
- net ~ON~: track 19.5 -> 0.00 mm
- net RX: track 13.6 -> 0.00 mm
- net TX: track 13.0 -> 0.00 mm
- net LED_W1_OUT: track 12.0 -> 0.00 mm
- net LED_W2_OUT: track 12.0 -> 0.00 mm
- net BOOT: track 11.4 -> 0.00 mm
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- removed copper zone on B.Cu, net +12V
- removed copper zone on B.Cu, net GND
- removed copper zone on F.Cu, net GND
- removed copper zone on B.Cu, net GNDPWR
- removed copper zone on F.Cu, net GNDPWR
Other:
- board outline removed
- board text removed: "DUMMY IO32"
- board text removed: "LED_W1 IO33"
- board text removed: "LED_W2 IO25"
- board text removed: "RGB1 IO26"
- board text removed: "RGB2 IO27"

Commit message: Finished.
Parts:
- removed C4, C6: 10u, Capacitor_SMD:C_1206_3216Metric_Pad1.42x1.75mm_HandSolder
- removed C5: 1u, Capacitor_SMD:C_1206_3216Metric_Pad1.42x1.75mm_HandSolder
- removed D4, D6: D_Schottky, Diode_SMD:D_SOD-323_HandSoldering
- removed D5: LED_AGRB, custom:LED_STRIP_RGB
- removed D7: LED, custom:LED_STRIP
- removed R7: 33k, Resistor_SMD:R_0805_2012Metric_Pad1.15x1.40mm_HandSolder
- removed R8, R9: 10k, Resistor_SMD:R_0805_2012Metric_Pad1.15x1.40mm_HandSolder
- added U3: TSOP343xx, OptoDevice:Vishay_MOLD-3Pin, F.Cu at (98.5, 93.2)
- C2: value 10u -> 1u; footprint Capacitor_SMD:C_1206_3216Metric_Pad1.42x1.75mm_HandSolder -> Capacitor_SMD:C_0805_2012Metric_Pad1.15x1.40mm_HandSolder
- C3: value 10u -> 22u
- D1: footprint Diode_SMD:D_SOD-323_HandSoldering -> Diode_SMD:D_SMA
- D2: value D_Schottky -> LED_AGRB; footprint Diode_SMD:D_SOD-323_HandSoldering -> custom:LED_STRIP_RGB
- D3: value D_Schottky -> LED; footprint Diode_SMD:D_SOD-323_HandSoldering -> custom:LED_STRIP
- J1: footprint Connector_FFC-FPC:Hirose_FH12-6S-0.5SH_1x06-1MP_P0.50mm_Horizontal -> Connector_JST:JST_SH_SM06B-SRSS-TB_1x06-1MP_P1.00mm_Horizontal; moved to B.Cu
- L1: value 6u5 -> 10u; footprint Inductor_SMD:L_Bourns-SRN4018 -> Inductor_SMD:L_Wuerth_MAPI-4020
- Q1, Q2, Q3, Q4: moved to F.Cu
- R1: value 10k -> 100k
- R2: value 10k -> 47k
- R3: value 10k -> 33k
- R4: value 100k -> 470
- R6: value 47k -> 10k; moved to B.Cu
- U1: value AP65111AWU -> AP65211AWU
- moved Q4 80.7 mm to (102.0, 106.5), turned to 270 degrees
- moved Q2 80.2 mm to (90.0, 106.5), turned to 270 degrees
- moved U2 78.9 mm to (93.0, 79.8)
- moved Q1 74.2 mm to (86.0, 106.5), turned to 270 degrees
- moved J1 73.2 mm to (83.0, 95.2), turned to 90 degrees
- moved Q3 66.9 mm to (82.0, 106.5), turned to 270 degrees
- moved J2 62.2 mm to (103.0, 78.0)
- moved J3 61.0 mm to (83.0, 78.0)
- moved D3 60.9 mm to (99.5, 111.0), turned to 180 degrees
- moved D2 58.3 mm to (87.2, 111.0), turned to 180 degrees
- moved C2 41.0 mm to (92.8, 77.0)
- moved C1 40.6 mm to (89.5, 82.8), turned to 180 degrees
- moved R5 36.6 mm to (92.8, 75.0), turned to 180 degrees
- moved C3 35.1 mm to (88.5, 76.2)
- moved D1 34.5 mm to (88.2, 89.0), turned to 270 degrees
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Connections:
- C2 pad 1: +12V -> Net-(C2-Pad1)
- C2 pad 2: GND -> Net-(C2-Pad2)
- C3 pad 1: +12V -> VDD
- D1 pad 2: LED_R_OUT -> +5V
- D3 pad 1: +12V -> Net-(D3-Pad1)
- D3 pad 2: LED_B_OUT -> +12V
- J1 pad 1: +5V -> GND
- J1 pad 2: BOOT -> +5V
- J1 pad 4: RX -> TX
- J1 pad 5: TX -> RX
- J1 pad 6: GND -> BOOT
- L1 pad 1: Net-(C5-Pad1) -> Net-(C2-Pad1)
- Q4 pad 3: Net-(D6-Pad2) -> Net-(D3-Pad1)
- R1 pad 1: +12V -> Net-(R1-Pad1)
- R1 pad 2: LED_R_OUT -> +12V
- R2 pad 1: +12V -> Net-(R2-Pad1)
- R2 pad 2: LED_G_OUT -> Net-(R2-Pad2)
- R3 pad 1: +12V -> VDD
- R3 pad 2: LED_B_OUT -> Net-(R2-Pad2)
- R4 pad 1: Net-(R4-Pad1) -> Net-(R2-Pad2)
- R4 pad 2: +12V -> Net-(R4-Pad2)
- R5 pad 1: +12V -> Net-(R4-Pad2)
- R5 pad 2: Net-(D6-Pad2) -> GND
- R6 pad 1: Net-(R6-Pad1) -> VDD
- R6 pad 2: Net-(R6-Pad2) -> EN
- U1 pad 1: +12V -> GND
- U1 pad 2: GND -> Net-(C2-Pad1)
- U1 pad 3: Net-(C5-Pad1) -> +12V
- U1 pad 4: Net-(C5-Pad2) -> Net-(R2-Pad1)
- U1 pad 5: Net-(R4-Pad1) -> Net-(R1-Pad1)
- U1 pad 6: Net-(R6-Pad1) -> Net-(C2-Pad2)
- U2 pad 10: LED_G -> (no net)
- U2 pad 11: LED_B -> (no net)
- U2 pad 12: Net-(U2-Pad12) -> (no net)
- U2 pad 13: Net-(U2-Pad13) -> LED_W
- U2 pad 14: Net-(U2-Pad14) -> IR
- U2 pad 16: Net-(U2-Pad16) -> LED_G
- U2 pad 17: Net-(U2-Pad17) -> (no net)
- U2 pad 18: Net-(U2-Pad18) -> (no net)
- U2 pad 19: Net-(U2-Pad19) -> (no net)
- U2 pad 20: Net-(U2-Pad20) -> (no net)
- U2 pad 21: Net-(U2-Pad21) -> (no net)
- U2 pad 22: Net-(U2-Pad22) -> (no net)
- U2 pad 23: Net-(U2-Pad23) -> LED_R
- U2 pad 24: Net-(U2-Pad24) -> LED_B
- U2 pad 26: Net-(U2-Pad26) -> (no net)
- U2 pad 27: Net-(U2-Pad27) -> (no net)
- U2 pad 28: Net-(U2-Pad28) -> (no net)
- U2 pad 29: Net-(U2-Pad29) -> (no net)
- U2 pad 30: Net-(U2-Pad30) -> (no net)
- U2 pad 31: Net-(U2-Pad31) -> (no net)
- U2 pad 32: Net-(U2-Pad32) -> (no net)
- U2 pad 33: Net-(U2-Pad33) -> (no net)
- U2 pad 36: Net-(U2-Pad36) -> (no net)
- U2 pad 37: Net-(U2-Pad37) -> (no net)
- U2 pad 39: (no net) -> GND
- U2 pad 4: Net-(U2-Pad4) -> (no net)
- U2 pad 5: Net-(U2-Pad5) -> (no net)
- U2 pad 6: Net-(U2-Pad6) -> (no net)
- U2 pad 7: Net-(U2-Pad7) -> (no net)
- U2 pad 8: LED_W -> (no net)
- U2 pad 9: LED_R -> (no net)
Routing:
- net +12V: track 0.00 -> 71.5 mm, vias 0 -> 2
- net VDD: track 0.00 -> 56.0 mm, vias 0 -> 1
- net EN: track 0.00 -> 40.6 mm
- net LED_G: track 0.00 -> 27.7 mm, vias 0 -> 1
- net LED_W: track 0.00 -> 25.1 mm, vias 0 -> 1
- net LED_B: track 0.00 -> 23.4 mm, vias 0 -> 1
- net TX: track 0.00 -> 23.0 mm
- net LED_R: track 0.00 -> 21.9 mm, vias 0 -> 1
- net RX: track 0.00 -> 20.0 mm
- net GND: track 0.00 -> 15.4 mm, vias 0 -> 2
- net Net-(R2-Pad1): track 0.00 -> 8.89 mm
- net +5V: track 0.00 -> 8.27 mm, vias 0 -> 1
- net IR: track 0.00 -> 7.80 mm
- net Net-(J1-PadMP): track 0.00 -> 7.60 mm
- net Net-(C2-Pad1): track 0.00 -> 5.06 mm
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- added copper zone on B.Cu, net GND
- added copper zone on F.Cu, net GND
Other:
- board outline added: 26 x 44 mm

Commit message: Removed temporary files
Connections:
- J1 pad MP: Net-(J1-PadMP) -> GND
Routing:
- net Net-(J1-PadMP): track 7.60 -> 0.00 mm
- net GND: track 15.4 -> 23.0 mm
