File: luna.sch (KiCad schematic (older format))
At the start: 32 parts, among them J1 Conn_01x06_MountingPin, J2 Conn_01x01, J3 Conn_01x01, Q1 DMN3404L, Q2 DMN3404L, Q3 DMN3404L, Q4 DMN3404L, U1 AP65111AWU, U2 ESP32-WROOM-32

Commit message: Finished.
Parts:
- removed C2, C4, C6: 10u, Capacitor_SMD:C_1206_3216Metric_Pad1.42x1.75mm_HandSolder, symbol Device:C
- removed D1, D2, D3, D6: D_Schottky, Diode_SMD:D_SOD-323_HandSoldering, symbol Device:D_Schottky
- removed R1, R2, R3, R5: 10k, Resistor_SMD:R_0805_2012Metric_Pad1.15x1.40mm_HandSolder, symbol Device:R
- removed U1: AP65111AWU, Package_TO_SOT_SMD:TSOT-23-6, symbol Regulator_Switching:AP65111AWU
- added R4: 470, Resistor_SMD:R_0805_2012Metric_Pad1.15x1.40mm_HandSolder, symbol Device:R
- added U1: AP65211AWU, Package_TO_SOT_SMD:TSOT-23-6, symbol custom:AP65211AWU
- added U3: TSOP343xx, OptoDevice:Vishay_MOLD-3Pin, symbol Interface_Optical:TSOP343xx
- C2: renamed from C5; footprint Capacitor_SMD:C_1206_3216Metric_Pad1.42x1.75mm_HandSolder -> Capacitor_SMD:C_0805_2012Metric_Pad1.15x1.40mm_HandSolder
- C3: value 10u -> 22u
- D1: renamed from D4; footprint Diode_SMD:D_SOD-323_HandSoldering -> Diode_SMD:D_SMA
- J1: footprint Connector_FFC-FPC:Hirose_FH12-6S-0.5SH_1x06-1MP_P0.50mm_Horizontal -> Connector_JST:JST_SH_SM06B-SRSS-TB_1x06-1MP_P1.00mm_Horizontal
- L1: value 6u5 -> 10u; footprint Inductor_SMD:L_Bourns-SRN4018 -> Inductor_SMD:L_Wuerth_MAPI-4020
- renumbered D5 to D2, D7 to D3, R4 to R1, R6 to R2, R7 to R3, R8 to R5, R9 to R6
Connections:
- net labels added: IR
- wire segments 122 -> 79
- no-connect marks 26 -> 25
Other:
- moved on the sheet: D3, R5

Commit message: Removed temporary files
Connections:
- net GND: now also J1.MP (MountPin)
- no-connect marks 25 -> 24
Changed lines of the file:
@@
 	-1   0    0    -1
 $EndComp
-NoConn ~ 950  1950
 Wire Wire Line
 	4400 1350 4900 1350
@@
 	0    1    1    0
 $EndComp
+$Comp
+L power:GND #PWR?
+U 1 1 5E55F075
+P 950 1950
+F 0 "#PWR?" H 950 1700 50  0001 C CNN
+F 1 "GND" H 955 1777 50  0000 C CNN
+F 2 "" H 950 1950 50  0001 C CNN
+F 3 "" H 950 1950 50  0001 C CNN
+	1    950  1950
+	-1   0    0    -1
+$EndComp
 $EndSCHEMATC
